File: packs/pcb-kicad/selftest/assets/esd_guard.kicad_pcb (KiCad board)
At the start: 2 copper layers, 30 x 15 mm, 3 parts, among them J1 USB_IN, J2 USB_OUT, U1 USBLC6-2SC6

Commit message: pcb-kicad, phases 2-4: schematic, router, fab limits, SPICE, enclosure fit
Five gates and the first bundled proposer, each gate qualified on the
baseline (10 of 10 with kicad-cli, ngspice and CadQuery present; the
tool gates read Skipped without them, as on CI).

Phase 2, the schematic. pcb.erc (kicad-cli sch erc, its exit code) and
pcb.parity (pcb drc --schematic-parity, the report's parity count with
the exit code held to agree), both established. The baseline gains
esd_guard.kicad_sch, written from KiCad's stock symbols with fixed
UUIDs by make_schematic.py, and every footprint on the board links to
its symbol. Controls: a label typed "D+" where every other says "DP"
(ERC: a label nothing else shares), and U1 pin 6 moved to D- on the
schematic with the board not updated (parity: a pad on the wrong net).

Phase 3, the router. pcb.autoroute, a proposer (established): pcbnew
exports a DSN in a Python that has it, Freerouting routes on one thread
with its analytics off, the session is imported onto a copy outside the
project, and only the routed board and a summary are recorded. The DRC
gates judge it once a person adopts it.

Phase 4, beyond the copper. pcb.fab_rules (sourced): JLCPCB's published
minimums, each quoted with the day read, as the staged board's only
custom rules. pcb.spice (established): one .meas of ngspice -b on the
project's deck against a band; the baseline deck is VBUS at the output
header under a 0.5 A step. pcb.enclosure_fit (established): kicad-cli's
STEP export against the enclosure's solid, OpenCascade's shared volume
and distance, in a child process.

What slipped through while building it:
- ERC on a host whose KiCad was never configured warned about every
  symbol's library, so the baseline would have passed on one machine
  and failed on another. The project's own sym-lib-table and
  fp-lib-table seal it, and the gates stage them.
- pcbnew.FootprintLoad leaves a footprint with no library name, which
  parity reads as a footprint the symbo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
Parts:
- J1, J2: footprint PinHeader_1x04_P2.54mm_Vertical -> Connector_PinHeader_2.54mm:PinHeader_1x04_P2.54mm_Vertical
- U1: footprint SOT-23-6 -> Package_TO_SOT_SMD:SOT-23-6
